File: hardware/controller/controller.kicad_sch (KiCad schematic)
At the start: 14 parts, among them J1 Conn_01x02_Pin, J2 Conn_01x02_Pin, J3 Conn_01x02_Pin, J4 Conn_01x02_Pin, J5 USB C Lipo Pins, J7 IMU (gnd/vdd side), J8 UWB, U1 ESP32-S3-DEVKITC-1-N8R8

Commit message: routing done
Parts:
- Listener Switch1: renamed from S1
- Power Switch1: renamed from S2
- USB C Lipo1: renamed from J5
- renumbered U1 to ESP32, J7 to IMU1, J8 to UWB1
Connections:
- net at ESP32.J1_1 (3V3), R1.2, R2.2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: now also IMU1.6 (Pin_6), UWB1.6 (Pin_6)
Changed lines of the file:
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@@
+	)
+	(junction
+		(at 270.51 170.18)
+		(diameter 0)
+		(color 0 0 0 0)
 	)
 	(junction
@@
 	)
 	(junction
+		(at 323.85 170.18)
+		(diameter 0)
+		(color 0 0 0 0)
+	)
+	(junction
 		(at 269.24 231.14)
 		(diameter 0)
@@
 	(wire
 		(pts
-			(xy 270.51 160.02) (xy 270.51 172.72)
+			(xy 270.51 160.02) (xy 270.51 170.18)
 		)
 		(stroke
@@
 	(wire
 		(pts
+			(xy 270.51 170.18) (xy 270.51 172.72)
+		)
+		(stroke
+			(width 0)
+			(type default)
+		)
+	)
+	(wire
+		(pts
 			(xy 321.31 182.88) (xy 321.31 185.42)
 		)
@@
 		(pts
 			(xy 261.62 226.06) (xy 261.62 231.14)
+		)
+		(stroke
+			(width 0)
+			(type default)
+		)
+	)
+	(wire
+		(pts
+			(xy 270.51 170.18) (xy 323.85 170.18)
 		)
 		(stroke
@@
 		(dnp no)
 		(fields_autoplaced yes)
-		(property "Reference" "U1"
+		(property "Reference" "ESP32"
 			(at 293.37 165.1 0)
 			(effects
@@
 			(project ""
 				(path "/50de191a-06b5-4968-8f0c-17f7744c4812"
-					(reference "U1")
+					(reference "ESP32")
 					(unit 1)
 				)
@@
 		(on_board yes)
 		(dnp no)
-		(property "Reference" "J7"
+		(property "Reference" "IMU1"
 			(at 336.042 215.646 0)
 			(effects
@@
 			(project "controller"
 				(path "/50de191a-06b5-4968-8f0c-17f7744c4812"
-					(reference "J7")
+					(reference "IMU1")
 					(unit 1)
 				)
@@
 		(on_board yes)
 		(dnp no)
-		(property "Reference" "J8"
+		(property "Reference" "UWB1"
 			(at 333.502 164.592 0)
 			(effects
@@
 			(project ""
 				(path "/50de191a-06b5-4968-8f0c-17f7744c4812"
-					(reference "J8")
+					(reference "UWB1")
 					(unit 1)
 				)
@@
 		(on_board yes)
 		(dnp no)
-		(property "Reference" "S2"
+		(property "Reference" "Power Switch1"
 			(at 276.86 240.538 90)
 			(effects
@@
 			(project ""
 				(path "/50de191a-06b5-4968-8f0c-17f7744c4812"
-					(reference "S2")
+					(reference "Power Switch1")
 					(unit 1)
 				)
@@
 		(dnp no)
 		(fields_autoplaced yes)
-		(property "Reference" "S1"
+		(property "Reference" "Listener Switch1"
 			(at 373.38 191.7714 90)
 			(effects
@@
 			(project ""
 				(path "/50de191a-06b5-4968-8f0c-17f7744c4812"
-					(reference "S1")
+					(reference "Listener Switch1")
 					(unit 1)
 				)
@@
 		(on_board yes)
 		(dnp no)
-		(property "Reference" "J5"
+		(property "Reference" "USB C Lipo1"
 			(at 262.89 263.144 90)
 			(effects
@@
 			(project ""
 				(path "/50de191a-06b5-4968-8f0c-17f7744c4812"
-					(reference "J5")
+					(reference "USB C Lipo1")
 					(unit 1)
 				)
